File: hardware/main_hw/bitdoglab_v5_3_smd/bitdoglab_smd.kicad_sch (KiCad schematic)
At the start: 154 parts, among them J1 Conn_01x03, J12 Conn_01x05_Pin, J19 JOYSTICK, J2 conector_idc, J20 Conn_01x04_Pin, J21 Conn_01x04_Pin, J3 Conn_01x03_Pin, J4 Conn_01x02, J5 Conn_01x05_Pin, J6 Conn_01x20_Socket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

Commit message: Atualização de projeto bitdoglab 5.3 e esquemáticos bitdoglab 5.3 e bitdoglab 6.2
Parts:
- removed C39, C40, C41: 0.1µF, Capacitor_SMD:C_0402_1005Metric, symbol Adafruit MAX4466 Mic Amp-altium-import:root_0_CAP_CERAMIC0805
- removed C42: 10u, Resistor_SMD:R_0805_2012Metric, symbol IP5306-LiPoChargerBooster_orcad-altium-import:0_10u
- removed J3: Conn_01x03_Pin, Connector_PinHeader_2.54mm:PinHeader_1x03_P2.54mm_Vertical, symbol Connector:Conn_01x03_Pin
- removed J4: Conn_01x02, Connector_PinHeader_2.54mm:PinHeader_1x02_P2.54mm_Vertical, symbol Connector_Generic:Conn_01x02
- removed J6, J7, J8, J9: Conn_01x20_Socket, Connector_PinSocket_2.54mm:PinSocket_1x20_P2.54mm_Vertical_SMD_Pin1Right, symbol Connector:Conn_01x20_Socket
- removed Q3, Q6: BSS138, Package_TO_SOT_SMD:SOT-23, symbol Transistor_FET:BSS138
- removed R10, R16, R20, R21, R22, R23, R9: 10k, Resistor_SMD:R_0603_1608Metric, symbol IP5306-LiPoChargerBooster_orcad-altium-import:2_10k
- removed R11, R15, R24, R25: 0R, Resistor_SMD:R_0603_1608Metric, symbol Device:R
- removed R17: 2.5K, Resistor_SMD:R_0603_1608Metric, symbol IP5306-LiPoChargerBooster_orcad-altium-import:2_10k
- removed R18: 5.32K, Resistor_SMD:R_0603_1608Metric, symbol IP5306-LiPoChargerBooster_orcad-altium-import:2_10k
- removed R19: 30.1K, Resistor_SMD:R_0603_1608Metric, symbol IP5306-LiPoChargerBooster_orcad-altium-import:2_10k
- removed R26, R27, R28, R29, R30, R31: 1K, Resistor_SMD:R_0603_1608Metric, symbol Adafruit MAX4466 Mic Amp-altium-import:root_1_RESISTOR0805
- removed U1: BQ25622ERYKR, Package_DFN_QFN:WQFN-HR18_RYK_TEX, symbol 2024-07-18_13-31-18:BQ25622ERYKR
- added C12, C13: 22u, Resistor_SMD:R_0805_2012Metric, symbol IP5306-LiPoChargerBooster_orcad-altium-import:0_22u
- added J3: Conn_01x02, Connector_PinHeader_2.54mm:PinHeader_1x02_P2.54mm_Vertical, symbol Connector_Generic:Conn_01x02
- added LED1: 25%, BITDOG_HWIT1:LED_0805_2012Metric, symbol IP5306-LiPoChargerBooster_orcad-altium-import:3_25%
- added LED2: 50%, BITDOG_HWIT1:LED_0805_2012Metric, symbol IP5306-LiPoChargerBooster_orcad-altium-import:1_50%
- added LED3: 75%, BITDOG_HWIT1:LED_0805_2012Metric, symbol IP5306-LiPoChargerBooster_orcad-altium-import:3_75%
- added R10, R9: 2R, Resistor_SMD:R_0603_1608Metric, symbol IP5306-LiPoChargerBooster_orcad-altium-import:1_2R
- added R11: 20R, Resistor_SMD:R_0603_1608Metric, symbol IP5306-LiPoChargerBooster_orcad-altium-import:2_20R
- added R15: 100R, Resistor_SMD:R_1210_3225Metric, symbol IP5306-LiPoChargerBooster_orcad-altium-import:2_10k
- added U3: IP5306, Package_SO:SOP-8_5.28x5.23mm_P1.27mm, symbol IP5306-LiPoChargerBooster_orcad-altium-import:0_IP5306
Connections:
- net GNDREF: now also C9.2, KEY1.2, LED5.2 (K), C12.2, C13.2, J3.2 (Pin_2), R15.2, U3.9 (EP); no longer KEY1.1
- net VBUS: now also C8.1, R9.2, U3.1 (VIN); no longer C7.1
- net V_BAT +: now also C9.1, L1.2, R10.2
- net at R12.1: now also KEY1.1; no longer KEY1.2
- net at L1.1: now also U3.7 (SW)
- net at C10.1: now also R10.1, U3.6 (BAT); no longer C9.1
- net at D28.2 (DOUT): now also J3.1 (Pin_1)
- net at LED4.2 (K): now also LED3.1 (A), U3.3 (LED2)
- net 3V3_EN renamed pino_37
- net BUZZER_A renamed pino_27
- net GP05 renamed pino_07
- net GP06 renamed pino_09
- net RUN renamed pino_30
- net SCL renamed pino_20
- net SDA renamed pino_19
- removed net VSYS_1: C11.1, L1.2, LED4.1 (A), LED5.1 (A), Q5.3 (D), R12.2
- new net: C11.1, C12.1, C13.1, Q5.3 (D), R15.1, U3.8 (VOUT)
- new net: LED1.1 (A), LED2.2 (K), U3.2 (LED1)
- new net: LED1.2 (K), LED2.1 (A), LED3.2 (K), LED4.1 (A), U3.4 (LED3)
- new net: C7.1, R9.1
- new net: R11.2, R12.2, U3.5 (KEY)
- new net: LED5.1 (A), R11.1
- no-connect marks 0 -> 2
Other:
- note added: "16V"
- note removed: "CONNECTOR_PICO"
- title: BitDogLab SMD version -> BitDogLab Main SMD version
- moved on the sheet: C10, C11, C7, C8, C9, D1, J2, KEY1, L1, LED4, LED5, Q5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
